File: posey-rx.kicad_sch (KiCad schematic)
At the start: 29 parts, among them J1 TC2050-IDC-NL, Y1 XTAL, Y2 XTAL

Commit message: Updated readme, license, and version.
Parts:
- added C10: 0.1µ, Capacitor_SMD:C_0402_1005Metric, symbol Device:C
- D1: value D_TVS -> ACPDQC5V0R-HF
- IMU1: value BNO080 -> BNO086
- J1, LiPo1, Vin1: now left out of the parts list
- R10, R12: now not fitted; now left out of the parts list
- TH1: value NTC -> 10k
- Y1, Y2: value XTAL -> ECS-.327-9-16-TR
Connections:
- net GND: now also C10.1; no longer IMU1.5 (PS1), IMU1.6 (PS0/WAKE)
- net SCL/SPI_SCK: now also µC1.18 (P0-11); no longer µC1.17 (P0-10)
- net SDA/SPI_CIPO: now also µC1.20 (P0-08); no longer µC1.18 (P0-11)
- net SPI_CS_IMU: now also µC1.42 (P0-19); no longer µC1.16 (P0-09)
- net VCC: now also C10.2
- new net IMU_PS0: IMU1.6 (PS0/WAKE), µC1.16 (P0-09)
- new net IMU_PS1: IMU1.5 (PS1), µC1.17 (P0-10)
Other:
- note removed: "2023.10.19"
- note removed: "2310"
- note removed: "Posey IMU Platform"
- note removed: "Soft Machines Lab Carnegie Mellon University License here"
- company: (none) -> Soft Machines Lab
- title: (none) -> Posey Ring
